File: photometric-leds.kicad_pcb (KiCad board)
At the start: 2 copper layers, 50 x 50 mm, 45 parts, among them J1 CONN_02X03, J2 CONN_02X03, U1 ATTINY20-SSU, U2 pam2800, U3 pam2800, U4 pam2800, U5 pam2800, U6 pam2800

Commit message: Added mechanical drawings
Parts:
- J2: footprint Connectors_Molex:Molex_Picoflex_90325_06x1.27mm_Straight -> Connectors_Molex:Molex_Picoflex_90814_06x1.27mm_Straight
- moved J2 3.64 mm to (149.5, 71.0)
Routing:
- net +5V: track 130.8 -> 195.7 mm
- net Net-(J2-Pad1): track 37.3 -> 68.6 mm
- net Net-(J1-Pad1): track 105.2 -> 90.1 mm
- net Net-(J1-Pad3): track 75.0 -> 66.6 mm
- net Net-(J1-Pad5): track 85.9 -> 80.3 mm
- net GND: track 290.3 -> 294.8 mm
- net (no net): track 0.00 -> 0.50 mm
Other:
- board size 50 x 50 mm -> 75 x 62.5 mm
