File: photometric-leds.sch (KiCad schematic (older format))
At the start: 45 parts, among them J1 CONN_02X03, J2 CONN_02X03, U1 ATTINY20-SSU, U2 pam2800, U3 pam2800, U4 pam2800, U5 pam2800, U6 pam2800

Commit message: Added mechanical drawings
Parts:
- C1, C2: symbol device:C -> Device:C
- J2: footprint Connectors_Molex:Molex_Picoflex_90325_06x1.27mm_Straight -> Connectors_Molex:Molex_Picoflex_90814_06x1.27mm_Straight
- MK1: symbol mechanical:Mounting_Hole_PAD -> Mechanical:MountingHole_Pad
- U1: symbol atmel:ATTINY20-SSU -> MCU_Microchip_ATtiny:ATtiny20-SSU
- U2, U3, U4, U5, U6: symbol local:pam2800 -> photometric-leds-rescue:pam2800-RESCUE-photometric-leds
Connections:
- wire segments 164 -> 186
Other:
- moved on the sheet: U1
Changed lines of the file:
@@
 $EndDescr
 $Comp
-L local:pam2800 U2
+L photometric-leds-rescue:pam2800-RESCUE-photometric-leds U2
 U 1 1 5A04D1B7
 P 9150 2000
@@
 	10700 1700 10700 2050
 Wire Wire Line
-	10350 2000 10350 2100
+	10350 2000 10350 2050
 Wire Wire Line
 	10700 2350 10700 2450
@@
 Connection ~ 10350 2050
 Wire Wire Line
-	10000 2100 10000 2000
+	10000 2100 10000 2050
 Wire Wire Line
 	9650 1700 9650 1800
-Connection ~ 10000 1700
 Wire Wire Line
 	9650 2000 9650 2050
@@
 $EndComp
 Wire Wire Line
-	8650 1800 8550 1800
+	8650 1800 8600 1800
 Wire Wire Line
 	8600 1800 8600 1750
@@
 	8150 1900 8650 1900
 $Comp
-L local:pam2800 U3
+L photometric-leds-rescue:pam2800-RESCUE-photometric-leds U3
 U 1 1 5A04E08E
 P 9150 2800
@@
 	10700 2500 10700 2850
 Wire Wire Line
-	9650 2500 10700 2500
-Wire Wire Line
-	10350 2800 10350 2900
+	10350 2800 10350 2850
 Wire Wire Line
 	10700 3150 10700 3250
@@
 Connection ~ 10350 2850
 Wire Wire Line
-	10000 2900 10000 2800
+	10000 2900 10000 2850
 Wire Wire Line
 	9650 2500 9650 2600
-Connection ~ 10000 2500
 Wire Wire Line
 	9650 2800 9650 2850
@@
 $EndComp
 Wire Wire Line
-	8650 2600 8550 2600
+	8650 2600 8600 2600
 Wire Wire Line
 	8600 2600 8600 2550
@@
 	8150 2700 8650 2700
 $Comp
-L local:pam2800 U4
+L photometric-leds-rescue:pam2800-RESCUE-photometric-leds U4
 U 1 1 5A04E92D
 P 9150 3600
@@
 	10700 3300 10700 3650
 Wire Wire Line
-	9650 3300 10700 3300
-Wire Wire Line
-	10350 3600 10350 3700
+	10350 3600 10350 3650
 Wire Wire Line
 	10700 3950 10700 4050
@@
 Connection ~ 10350 3650
 Wire Wire Line
-	10000 3700 10000 3600
+	10000 3700 10000 3650
 Wire Wire Line
 	9650 3300 9650 3400
-Connection ~ 10000 3300
 Wire Wire Line
 	9650 3600 9650 3650
@@
 $EndComp
 Wire Wire Line
-	8650 3400 8550 3400
+	8650 3400 8600 3400
 Wire Wire Line
 	8600 3400 8600 3350
@@
 	8150 3400 8150 3500
 $Comp
-L local:pam2800 U5
+L photometric-leds-rescue:pam2800-RESCUE-photometric-leds U5
 U 1 1 5A04E97A
 P 9150 4400
@@
 	10700 4100 10700 4450
 Wire Wire Line
-	9650 4100 10700 4100
-Wire Wire Line
-	10350 4400 10350 4500
+	10350 4400 10350 4450
 Wire Wire Line
 	10700 4750 10700 4850
@@
 Connection ~ 10350 4450
 Wire Wire Line
-	10000 4500 10000 4400
+	10000 4500 10000 4450
 Wire Wire Line
 	9650 4100 9650 4200
-Connection ~ 10000 4100
 Wire Wire Line
 	9650 4400 9650 4450
@@
 $EndComp
 Wire Wire Line
-	8650 4200 8550 4200
+	8650 4200 8600 4200
 Wire Wire Line
 	8600 4200 8600 4150
@@
 	8150 4300 8650 4300
 $Comp
-L local:pam2800 U6
+L photometric-leds-rescue:pam2800-RESCUE-photometric-leds U6
 U 1 1 5A04EC24
 P 9150 5200
@@
 	10700 4900 10700 5250
 Wire Wire Line
-	9650 4900 10700 4900
-Wire Wire Line
-	10350 5200 10350 5300
+	10350 5200 10350 5250
 Wire Wire Line
 	10700 5550 10700 5650
@@
 Connection ~ 10350 5250
 Wire Wire Line
-	10000 5300 10000 5200
+	10000 5300 10000 5250
 Wire Wire Line
 	9650 4900 9650 5000
-Connection ~ 10000 4900
 Wire Wire Line
 	9650 5200 9650 5250
@@
 $EndComp
 Wire Wire Line
-	8650 5000 8550 5000
+	8650 5000 8600 5000
 Wire Wire Line
 	8600 5000 8600 4950
@@
 F 0 "J2" H 6200 3050 50  0000 C CNN
 F 1 "CONN_02X03" H 6200 2650 50  0000 C CNN
-F 2 "Connectors_Molex:Molex_Picoflex_90325_06x1.27mm_Straight" H 6200 1650 50  0001 C CNN
+F 2 "Connectors_Molex:Molex_Picoflex_90814_06x1.27mm_Straight" H 6200 1650 50  0001 C CNN
 F 3 "" H 6200 1650 50  0001 C CNN
 	1    6200 2850
@@
 $EndComp
 Wire Wire Line
-	6500 2700 6500 2850
+	6500 2700 6500 2750
 Wire Wire Line
 	6500 2850 6450 2850
@@
 	6500 2950 6500 3150
 Wire Wire Line
-	6500 3150 5900 3150
+	6500 3150 6200 3150
 Wire Wire Line
 	5900 3150 5900 2950
@@
 $EndComp
 $Comp
-L device:C C2
+L Device:C C2
 U 1 1 5A0545A7
 P 2750 3150
@@
 $EndComp
 $Comp
-L device:C C1
+L Device:C C1
 U 1 1 5A054614
 P 2550 3150
@@
 	5300 4150 5300 4100
 $Comp
-L atmel:ATTINY20-SSU U1
+L MCU_Microchip_ATtiny:ATtiny20-SSU U1
 U 1 1 5A0674A9
 P 4100 3150
@@
 	5300 3800 5300 3750
 Wire Wire Line
-	5250 3750 5950 3750
+	5250 3750 5300 3750
 Connection ~ 5300 3750
 Wire Wire Line
-	5250 3550 5950 3550
+	5250 3550 5850 3550
 Wire Wire Line
 	5950 3650 5750 3650
@@
 Wire Wire Line
 	5450 2750 5250 2750
-Wire Wire Line
-	9650 1700 10700 1700
-Connection ~ 10350 1700
-Connection ~ 10350 2500
-Connection ~ 10350 3300
-Connection ~ 10350 4100
-Connection ~ 10350 4900
-$Comp
-L mechanical:Mounting_Hole_PAD MK1
+$Comp
+L Mechanical:MountingHole_Pad MK1
 U 1 1 5A06C830
 P 3050 4750
@@
 $EndComp
 Wire Wire Line
-	3050 4950 3050 4850
+	3050 4950 3050 4900
 Wire Wire Line
 	3300 4850 3300 4900
 Wire Wire Line
-	3050 4900 3800 4900
+	3050 4900 3300 4900
 Connection ~ 3050 4900
 Wire Wire Line
@@
 	3800 4900 3800 4850
 Connection ~ 3550 4900
+Wire Wire Line
+	10350 2050 10350 2100
+Wire Wire Line
+	10000 2050 10000 2000
+Wire Wire Line
+	8600 1800 8550 1800
+Wire Wire Line
+	10350 2850 10350 2900
+Wire Wire Line
+	10000 2850 10000 2800
+Wire Wire Line
+	8600 2600 8550 2600
+Wire Wire Line
+	10350 3650 10350 3700
+Wire Wire Line
+	10000 3650 10000 3600
+Wire Wire Line
+	8600 3400 8550 3400
+Wire Wire Line
+	10350 4450 10350 4500
+Wire Wire Line
+	10000 4450 10000 4400
+Wire Wire Line
+	8600 4200 8550 4200
+Wire Wire Line
+	10350 5250 10350 5300
+Wire Wire Line
+	10000 5250 10000 5200
+Wire Wire Line
+	8600 5000 8550 5000
+Wire Wire Line
+	6500 2750 6500 2850
+Wire Wire Line
+	6200 3150 5900 3150
+Wire Wire Line
+	5300 3750 5950 3750
+Wire Wire Line
+	5850 3550 5950 3550
+Wire Wire Line
+	3050 4900 3050 4850
+Wire Wire Line
+	3300 4900 3550 4900
+Wire Wire Line
+	3550 4900 3800 4900
+Wire Wire Line
+	9650 1700 10700 1700
+Wire Wire Line
+	9650 2500 10700 2500
+Wire Wire Line
+	9650 3300 10700 3300
+Wire Wire Line
+	9650 4100 10700 4100
+Wire Wire Line
+	9650 4900 10700 4900
 $EndSCHEMATC
